File: PCB/UwUstatus/UwUstatus.kicad_sch (KiCad schematic)
At the start: 8 parts, among them J1 Conn_01x15, J2 Conn_01x02, J3 Conn_01x06, U2 L7805

Commit message: Final revision
Parts:
- U2: footprint Package_TO_SOT_SMD:SOT-223-3_TabPin2 -> Package_TO_SOT_SMD:TO-252-2
Changed lines of the file:
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@@
 			)
 		)
-		(property "Footprint" "Package_TO_SOT_SMD:SOT-223-3_TabPin2"
+		(property "Footprint" "Package_TO_SOT_SMD:TO-252-2"
 			(at 74.295 26.67 0)
 			(effects
